Commit message: 仿真方案已经完备，只需要运行ros2 launch v550_navigation simulation_nav.launch.py 即可

File: src/wheeltec_robot_urdf/wheeltec_robot_urdf/urdf/V550_mec_robot.urdf (robot description, URDF)
Before this commit: robot V550_mec_robot, 8 links, 7 joints
Joints:
- joint laser_joint: origin xyz=0.0834767944381037 1.32296970929568E-05 0.09655 rpy=0 0 -3.14159265358979 -> xyz=0.0834767944381037 1.32296970929568E-05 0.09655 rpy=0 0 0
